File: KiCad/Timer_PCB/Timer_PCB.kicad_sch (KiCad schematic)
At the start: 4 parts, among them M1 Stepper_Motor_unipolar_5pin

Commit message: mise à jour du fichier kicad
Parts:
- added C1: 0.01, Capacitor_THT:C_Disc_D3.0mm_W2.0mm_P2.50mm, symbol PCM_SL_Devices:Capacitor_NP
- added D2, D3, D4, D5, D6, D7, D8, D9: WS2812, LED_SMD:LED_WS2812_PLCC6_5.0x5.0mm_P1.6mm, symbol LED:WS2812
- added SW1, SW2, SW3, SW4: SW_SPDT, symbol Switch:SW_SPDT
- added U1: ULN2003, symbol Transistor_Array:ULN2003
- added condensateur2: 1e-7, Capacitor_THT:C_Disc_D3.0mm_W2.0mm_P2.50mm, symbol PCM_SL_Devices:Capacitor_NP
Connections:
- net at BT1.1 (+), U2.15 (3V): now also D1.5 (VDD), D2.5 (VDD), D3.5 (VDD), D4.5 (VDD), D5.5 (VDD), D6.5 (VDD), D7.5 (VDD), D8.5 (VDD), D9.5 (VDD)
- net at U2.17 (GPIO33): now also D1.2 (DIN)
- net at U2.21 (GPIO38): now also BT1.2 (-), D1.6 (VSS), U2.29 (GND), U2.30 (GND), D2.6 (VSS), D3.6 (VSS), D4.6 (VSS), D5.6 (VSS), D6.6 (VSS), D7.6 (VSS), D8.6 (VSS), D9.6 (VSS), SW1.2 (B), SW2.2 (B), SW3.2 (B), SW4.2 (B), SW4.3 (C)
- net at U2.22 (GPIO36): now also SW4.1 (A)
- net at U2.23 (GPIO34): now also SW3.3 (C)
- net at U2.24 (GPIO35): now also SW3.1 (A); no longer D1.2 (DIN)
- net at U2.25 (GPIO21): now also SW2.3 (C)
- net at U2.26 (GPIO18): now also SW2.1 (A)
- net at U2.27 (GPIO17): now also SW1.3 (C)
- net at U2.28 (GPIO16): now also SW1.1 (A)
- net strapping pin: now reaches U2.4 (GPIO3)
- net at M1.1: now also M1.2, M1.3 (-), U1.14 (O3), U1.15 (O2), U1.16 (O1)
- net at M1.4: now also U1.13 (O4)
- net at M1.5: now also U1.12 (O5)
- net at D1.1 (DOUT): now also D2.2 (DIN)
- new net: D6.1 (DOUT), D7.2 (DIN)
- new net: D5.1 (DOUT), D6.2 (DIN)
- new net: D3.1 (DOUT), D4.2 (DIN)
- new net: D2.1 (DOUT), D3.2 (DIN)
- new net: D4.1 (DOUT), D5.2 (DIN)
- new net: D7.1 (DOUT), D8.2 (DIN)
- new net: D8.1 (DOUT), D9.2 (DIN)
Other:
- moved on the sheet: D1, M1
